File: eagle/mini_exp_v1-1-0a.brd (EAGLE design)
At the start: 208.6 x 112.5 mm, 30 parts, among them J1 CR22A-44D-2.54DS(70)STRAIGHT, J2 CR22A-44D-2.54DS(70)STRAIGHT, J3 DB9-MALE-RA, J4 DB9-MALE-RA, U1 AY-3-8910, U2 74LS244N, U3 74LS244N, U4 74LS74N, U5 74LS30N, U6 74LS04N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

Commit message: Post PCB check edits
Parts:
- moved J3 0.05 mm to (10.2, 56.0)
Routing:
- net N$14: track 0.00 -> 5.21 mm
- net N$15: track 0.00 -> 4.49 mm
- net N$171: track 1.37 -> 0.00 mm
- net N$169: track 1.35 -> 0.00 mm
- net N$165: track 1.29 -> 0.00 mm
- net N$163: track 1.22 -> 0.00 mm
- net N$167: track 1.17 -> 0.00 mm
- net N$170: track 0.92 -> 0.00 mm
- net N$18: track 57.0 -> 57.8 mm
- net GND: track 358.8 -> 359.4 mm
- net SND: track 196.1 -> 196.8 mm
- net DE01: track 210.1 -> 210.8 mm
- net !M1: track 155.7 -> 156.3 mm
- net IN-A15: track 34.0 -> 34.6 mm
- net IN-A12: track 58.7 -> 59.3 mm
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Other:
- outline, holes or cut-outs redrawn
- board text added: "Aquarius Mini Expander v1-1-0 Rev B - 02 SEP 2020 by Sean Harrington, sph@1stage.com"
- board text removed: "Aquarius Mini Expander v1-1-0 Rev A - 26 AUG 2020 by Sean Harrington, sph@1stage.com"
