File: eagle/mini_exp_v1-1-0b.brd (EAGLE design)
At the start: 208.6 x 112.5 mm, 30 parts, among them J1 CR22A-44D-2.54DS(70)STRAIGHT, J2 CR22A-44D-2.54DS(70)STRAIGHT, J3 DB9-MALE-RA, J4 DB9-MALE-RA, U1 AY-3-8910, U2 74LS244N, U3 74LS244N, U4 74LS74N, U5 74LS30N, U6 74LS04N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

Commit message: Clean up, post PCB arrival
Parts:
- added SJ1, SJ2: (no value), jumper:SJ
Connections:
- new net N$16: J1.P$44, SJ1.1
- new net N$17: J2.P$34, SJ2.1
- net GND: now also SJ1.2, SJ2.2; no longer J1.P$44, J2.P$34
Routing:
- net GND: track 359.4 -> 335.8 mm
- net N$17: track 0.00 -> 22.3 mm
- net N$16: track 0.00 -> 5.71 mm
Other:
- board text added: "Enable FRONT slot as RAM"
- board text added: "Enable REAR slot as ROM"
Changed lines of the file:
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@@
 <circle x="10.1854" y="68.58" radius="1.5748" width="0.0254" layer="20"/>
 <circle x="10.1854" y="43.5864" radius="1.5748" width="0.0254" layer="20"/>
+<text x="63.754" y="94.742" size="1.016" layer="21" rot="R270" align="center-left">Enable REAR slot as ROM</text>
+<text x="94.615" y="94.742" size="1.016" layer="21" rot="R270" align="center-left">Enable FRONT slot as RAM</text>
 </plain>
 <attributes>
@@
 <element name="XX02" library="aquarius" package="AQ-MX-BODGE-2" value="AQ-MX-BODGE-2" x="129.54" y="40.64" smashed="yes"/>
 <element name="XX03" library="aquarius" package="AQ-MX-BODGE-3" value="AQ-MX-BODGE-3" x="125.476" y="54.1274" smashed="yes"/>
+<element name="SJ1" library="jumper" library_urn="urn:adsk.eagle:library:252" package="SJ" package3d_urn="urn:adsk.eagle:package:15471/1" value="" x="94.615" y="96.647" smashed="yes" rot="R180">
+<attribute name="POPULARITY" value="33" x="94.615" y="96.647" size="1.778" layer="27" rot="R180" display="off"/>
+<attribute name="VALUE" x="94.2149" y="96.647" size="0.02" layer="27" rot="R180"/>
+</element>
+<element name="SJ2" library="jumper" library_urn="urn:adsk.eagle:library:252" package="SJ" package3d_urn="urn:adsk.eagle:package:15471/1" value="" x="63.754" y="96.393" smashed="yes">
+<attribute name="POPULARITY" value="33" x="63.754" y="96.393" size="1.778" layer="27" display="off"/>
+<attribute name="VALUE" x="64.1541" y="96.393" size="0.02" layer="27"/>
+</element>
 </elements>
 <signals>
@@
 <vertex x="137.704690625" y="93.39208125"/>
 <vertex x="134.77738125" y="96.04916875"/>
-<vertex x="97.938259375" y="96.04916875"/>
-<vertex x="96.29451875" y="94.40543125"/>
+<vertex x="97.674709375" y="96.04916875"/>
+<vertex x="97.155" y="97.79"/>
+<vertex x="97.1169" y="98.171"/>
+<vertex x="94.234" y="98.171"/>
+<vertex x="94.234" y="94.488"/>
+<vertex x="96.29451875" y="92.42748125"/>
 <vertex x="96.29451875" y="84.56513125"/>
 <vertex x="98.85031875" y="82.00933125"/>
@@
 <vertex x="74.084590625" y="70.228840625"/>
 <vertex x="65.527859375" y="78.78558125"/>
-<vertex x="65.527859375" y="93.07683125"/>
-<vertex x="62.165209375" y="96.43948125"/>
-<vertex x="53.698540625" y="96.43948125"/>
+<vertex x="65.527859375" y="95.762140625"/>
+<vertex x="63.58051875" y="97.70948125"/>
+<vertex x="61.76848125" y="97.70948125"/>
+<vertex x="60.956528125" y="96.897528125"/>
+<vertex x="53.698540625" y="96.94748125"/>
 <vertex x="53.698540625" y="94.998340625"/>
 <vertex x="51.665159375" y="94.998340625"/>
@@
 <contactref element="U1" pad="1"/>
 <contactref element="J1" pad="P$34"/>
-<contactref element="J1" pad="P$44"/>
 <contactref element="C9" pad="1"/>
 <contactref element="C10" pad="1"/>
@@
 <contactref element="C1" pad="2"/>
 <contactref element="R3" pad="2"/>
-<contactref element="J2" pad="P$34"/>
-<contactref element="J2" pad="P$44"/>
 <contactref element="C7" pad="1"/>
 <contactref element="C4" pad="1"/>
@@
 <vertex x="9.80398125" y="3.78651875"/>
 </polygon>
-<wire x1="100.1522" y1="94.3864" x2="100.1522" y2="96.3422" width="0.6096" layer="16"/>
-<wire x1="100.1522" y1="96.3422" x2="100.33" y2="96.52" width="0.6096" layer="16"/>
 <wire x1="55.3212" y1="6.0452" x2="59.4614" y2="1.905" width="0.6096" layer="16"/>
 <wire x1="59.4614" y1="1.905" x2="91.9734" y2="1.905" width="0.6096" layer="16"/>
@@
 <wire x1="157.48" y1="45.72" x2="157.9626" y2="45.72" width="0.6096" layer="16"/>
 <wire x1="165.6334" y1="47.9806" x2="165.7604" y2="47.8536" width="0.6096" layer="16"/>
-<wire x1="53.213" y1="81.5848" x2="52.9082" y2="81.28" width="0.6096" layer="16"/>
-<wire x1="52.9082" y1="81.28" x2="49.53" y2="81.28" width="0.6096" layer="16"/>
-<wire x1="49.53" y1="81.28" x2="48.26" y2="82.55" width="0.6096" layer="16"/>
-<wire x1="49.8348" y1="94.2848" x2="53.213" y2="94.2848" width="0.6096" layer="16"/>
-<wire x1="48.26" y1="82.55" x2="48.26" y2="92.71" width="0.6096" layer="16"/>
-<wire x1="48.26" y1="92.71" x2="49.8348" y2="94.2848" width="0.6096" layer="16"/>
 <wire x1="148.209" y1="70.6374" x2="151.4856" y2="70.6374" width="0.6096" layer="16"/>
 <wire x1="153.924" y1="68.199" x2="155.9306" y2="68.199" width="0.6096" layer="16"/>
@@
 <via x="17.1704" y="43.5864" extent="1-16" drill="1" diameter="1.3"/>
 <via x="17.1704" y="39.5986" extent="1-16" drill="1" diameter="1.3"/>
+<contactref element="SJ1" pad="2"/>
+<contactref element="J2" pad="P$44"/>
+<contactref element="SJ2" pad="2"/>
 <wire x1="129.54" y1="35.56" x2="129.54" y2="48.26" width="0" layer="19" extent="1-1"/>
 <wire x1="182.0418" y1="81.5848" x2="187.8584" y2="91.5924" width="0" layer="19" extent="1-1"/>
@@
 <wire x1="25.273" y1="67.183" x2="25.781" y2="67.183" width="0.6096" layer="1"/>
 <wire x1="25.273" y1="67.183" x2="23.7236" y2="68.7324" width="0.6096" layer="1"/>
-<wire x1="14.11311875" y1="68.7324" x2="23.7236" y2="68.7324" width="0.6096" layer="1"/>
+<wire x1="14.24011875" y1="68.7324" x2="23.7236" y2="68.7324" width="0.6096" layer="1"/>
 <via x="17.8816" y="101.346" extent="1-16" drill="1" diameter="1.3"/>
 <wire x1="17.1704" y1="92.2528" x2="17.1704" y2="100.6348" width="0.6096" layer="16"/>
 <wire x1="17.1704" y1="100.6348" x2="17.8816" y2="101.346" width="0.6096" layer="16"/>
-<wire x1="11.34451875" y1="71.501" x2="14.11311875" y2="68.7324" width="0.6096" layer="1"/>
+<wire x1="11.47151875" y1="71.501" x2="14.24011875" y2="68.7324" width="0.6096" layer="1"/>
 <wire x1="7.0866" y1="74.60908125" x2="10.19468125" y2="71.501" width="0.6096" layer="1"/>
-<wire x1="10.19468125" y1="71.501" x2="11.34451875" y2="71.501" width="0.6096" layer="1"/>
+<wire x1="10.19468125" y1="71.501" x2="11.47151875" y2="71.501" width="0.6096" layer="1"/>
 <wire x1="7.0866" y1="90.3986" x2="7.0866" y2="74.60908125" width="0.6096" layer="1"/>
 </signal>
@@
 <wire x1="116.967" y1="10.922" x2="116.967" y2="12.065" width="0.254" layer="16"/>
 </signal>
+<signal name="N$16">
+<contactref element="J1" pad="P$44"/>
+<contactref element="SJ1" pad="1"/>
+<wire x1="100.1522" y1="94.3864" x2="97.6376" y2="94.3864" width="0.6096" layer="1"/>
+<wire x1="97.6376" y1="94.3864" x2="95.377" y2="96.647" width="0.6096" layer="1"/>
+</signal>
+<signal name="N$17">
+<contactref element="J2" pad="P$34"/>
+<contactref element="SJ2" pad="1"/>
+<wire x1="53.213" y1="81.5848" x2="55.88" y2="84.2518" width="0.6096" layer="1"/>
+<wire x1="62.865" y1="96.266" x2="62.992" y2="96.393" width="0.6096" layer="1"/>
+<wire x1="62.865" y1="96.266" x2="57.023" y2="96.266" width="0.6096" layer="1"/>
+<wire x1="55.88" y1="84.2518" x2="55.88" y2="95.123" width="0.6096" layer="1"/>
+<wire x1="55.88" y1="95.123" x2="57.023" y2="96.266" width="0.6096" layer="1"/>
+</signal>
 </signals>

Commit message: Added Control Pad interface boards, updated board PDF, updated schematic PDF
Parts:
- added JP1, JP2: (no value), aquarius2:1X10
- C9: value 10n -> 10nF
- Q1: value (none) -> 2N3904; device aq-transistor:TO92L -> aq-transistor:TO92
- moved Q1 0.46 mm to (35.6, 18.8), turned to 0 degrees
Connections:
- new net CPA-D00: JP1.5
- new net CPA-D01: JP1.4
- new net CPA-D02: JP1.2
- new net CPA-D03: JP1.1
- new net CPA-D04: JP1.6
- new net CPA-D05: JP1.8
- new net CPA-D06: JP1.10
- new net CPA-D07: JP1.9
- new net CPA-GND: JP1.3, JP1.7
- new net CPB-D00: JP2.5
- new net CPB-D01: JP2.4
- new net CPB-D02: JP2.2
- new net CPB-D03: JP2.1
- new net CPB-D04: JP2.6
- new net CPB-D05: JP2.8
- new net CPB-D06: JP2.10
- new net CPB-D07: JP2.9
- new net CPB-GND: JP2.3, JP2.7
- net CHABC: now also Q1.3; no longer Q1.1
- net SND: now also Q1.1; no longer Q1.3
Routing:
- net CPB-GND: track 0.00 -> 5.77 mm, vias 0 -> 1
- net CPA-GND: track 0.00 -> 5.73 mm, vias 0 -> 1
- net CPB-D07: track 0.00 -> 5.54 mm, vias 0 -> 1
- net CPB-D06: track 0.00 -> 5.54 mm, vias 0 -> 1
- net CPB-D05: track 0.00 -> 5.54 mm, vias 0 -> 1
- net CPB-D03: track 0.00 -> 5.52 mm, vias 0 -> 1
- net CPB-D01: track 0.00 -> 5.52 mm, vias 0 -> 1
- net CPB-D04: track 0.00 -> 5.52 mm, vias 0 -> 1
- net CPB-D02: track 0.00 -> 5.52 mm, vias 0 -> 1
- net CPB-D00: track 0.00 -> 5.52 mm, vias 0 -> 1
- net CPA-D07: track 0.00 -> 5.48 mm, vias 0 -> 1
- net CPA-D05: track 0.00 -> 5.48 mm, vias 0 -> 1
- net CPA-D04: track 0.00 -> 5.48 mm, vias 0 -> 1
- net CPA-D02: track 0.00 -> 5.48 mm, vias 0 -> 1
- net CPA-D01: track 0.00 -> 5.48 mm, vias 0 -> 1
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- added copper zone on layer 1, net CPA-GND
- added copper zone on layer 16, net CPA-GND
- added copper zone on layer 1, net CPB-GND
- added copper zone on layer 16, net CPB-GND
Other:
- outline, holes or cut-outs redrawn
- board text added: "09 SEP 2020"
- board text added: "Aquarius Mini Expander v1-1-0 - REV B"
- board text added: "Aquarius Mini Expander v1-1-0 Rev B - 09 SEP 2020 by Sean Harrington, sph@1stage.com"
- board text added: "Control Pad Interface Board"
- board text added: "Email"
- board text added: "Engineer"
- board text added: "Project"
- board text added: "Revision Date"
- board text added: "Sean P. Harrington"
- board text added: "Website"
- board text added: "aquarius.1stage.com"
- board text added: "sph@1stage.com"
- board text removed: "Aquarius Mini Expander v1-1-0 Rev B - 02 SEP 2020 by Sean Harrington, sph@1stage.com"
