File: eagle/mini_exp_v1-1-0b.sch (EAGLE design)
At the start: 30 parts, among them J1 CR22A-44D-2.54DS(70)STRAIGHT, J2 CR22A-44D-2.54DS(70)STRAIGHT, J3 DB9-MALE-RA, J4 DB9-MALE-RA, U1 AY-3-8910, U2 74LS244N, U3 74LS244N, U4 74LS74N, U5 74LS30N, U6 74LS04N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

Commit message: Clean up, post PCB arrival
Parts:
- added SJ1, SJ2: (no value), jumper:SJ
Connections:
- new net N$16: J1.X44, SJ1.1
- new net N$17: J2.X34, SJ2.1
- net GND: now also SJ1.2, SJ2.2; no longer J1.X44, J2.X34
Other:
- note added: "02 SEP 2020"
- note added: "Aquarius Mini Expander v1-1-0 - REV B"
- note added: "Front RAM enable"
- note added: "Rear ROM enable"
- note removed: "26 AUG 2020"
- note removed: "Aquarius Mini Expander v1-1-0 - REV A"
Changed lines of the file:
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@@
 <part name="XX03" library="aquarius" deviceset="AQ-MX-BODGE-3" device=""/>
 <part name="P+6" library="supply1" library_urn="urn:adsk.eagle:library:371" deviceset="VCC" device=""/>
+<part name="SJ1" library="jumper" library_urn="urn:adsk.eagle:library:252" deviceset="SJ" device="" package3d_urn="urn:adsk.eagle:package:15471/1"/>
+<part name="SJ2" library="jumper" library_urn="urn:adsk.eagle:library:252" deviceset="SJ" device="" package3d_urn="urn:adsk.eagle:package:15471/1"/>
+<part name="GND10" library="supply1" library_urn="urn:adsk.eagle:library:371" deviceset="GND" device=""/>
+<part name="GND11" library="supply1" library_urn="urn:adsk.eagle:library:371" deviceset="GND" device=""/>
 </parts>
 <sheets>
@@
 <text x="-106.68" y="-10.16" size="2.54" layer="97" align="center">Address Buffer</text>
 <text x="-101.6" y="96.52" size="2.54" layer="97" align="center">Balance/Filter Capacitors</text>
-<text x="-101.6" y="-111.76" size="2.54" layer="97" align="center">Aquarius Mini Expander v1-1-0 - REV A</text>
+<text x="-101.6" y="-111.76" size="2.54" layer="97" align="center">Aquarius Mini Expander v1-1-0 - REV B</text>
 <text x="-101.6" y="-106.68" size="2.54" layer="97" align="center">Project</text>
 <wire x1="-134.62" y1="-114.3" x2="-134.62" y2="-109.22" width="0.1524" layer="97"/>
@@
 <wire x1="-68.58" y1="-114.3" x2="-134.62" y2="-114.3" width="0.1524" layer="97"/>
 <wire x1="-134.62" y1="-109.22" x2="-68.58" y2="-109.22" width="0.1524" layer="97"/>
-<text x="-43.18" y="-111.76" size="2.54" layer="97" align="center">26 AUG 2020</text>
+<text x="-43.18" y="-111.76" size="2.54" layer="97" align="center">02 SEP 2020</text>
 <text x="-43.18" y="-106.68" size="2.54" layer="97" align="center">Revision Date</text>
 <wire x1="-68.58" y1="-114.3" x2="-68.58" y2="-109.22" width="0.1524" layer="97"/>
@@
 <text x="58.42" y="-106.68" size="2.54" layer="97" align="center">Email</text>
 <text x="58.42" y="-111.76" size="2.54" layer="97" align="center">sph@1stage.com</text>
+<text x="152.4" y="-38.1" size="2.54" layer="97" align="center">Front RAM enable</text>
+<text x="193.04" y="-38.1" size="2.54" layer="97" align="center">Rear ROM enable</text>
 </plain>
 <instances>
@@
 <instance part="P+6" gate="VCC" x="-68.58" y="-5.08" smashed="yes" rot="R90">
 <attribute name="VALUE" x="-66.04" y="-7.62" size="1.778" layer="96" rot="R180"/>
+</instance>
+<instance part="SJ1" gate="1" x="157.48" y="-27.94" smashed="yes" rot="R270">
+<attribute name="NAME" x="160.02" y="-25.4" size="1.778" layer="95" rot="R270"/>
+<attribute name="VALUE" x="153.67" y="-25.4" size="1.778" layer="96" rot="R270"/>
+</instance>
+<instance part="SJ2" gate="1" x="180.34" y="-27.94" smashed="yes" rot="R270">
+<attribute name="NAME" x="182.88" y="-25.4" size="1.778" layer="95" rot="R270"/>
+<attribute name="VALUE" x="176.53" y="-25.4" size="1.778" layer="96" rot="R270"/>
+</instance>
+<instance part="GND10" gate="1" x="165.1" y="-33.02" smashed="yes" rot="R90">
+<attribute name="VALUE" x="167.64" y="-35.56" size="1.778" layer="96" rot="R90"/>
+</instance>
+<instance part="GND11" gate="1" x="198.12" y="-33.02" smashed="yes" rot="R90">
+<attribute name="VALUE" x="200.66" y="-35.56" size="1.778" layer="96" rot="R90"/>
 </instance>
 </instances>
@@
 <net name="GND" class="0">
 <segment>
-<pinref part="J1" gate="G$1" pin="X44"/>
-<wire x1="165.1" y1="-22.86" x2="134.62" y2="-22.86" width="0.1524" layer="91"/>
-<pinref part="J2" gate="G$1" pin="X44"/>
-<wire x1="165.1" y1="-22.86" x2="187.96" y2="-17.78" width="0.1524" layer="91"/>
-<junction x="165.1" y="-22.86"/>
 <pinref part="GND3" gate="1" pin="GND"/>
 <wire x1="134.62" y1="-25.4" x2="134.62" y2="-22.86" width="0.1524" layer="91"/>
 <pinref part="J1" gate="G$1" pin="X34"/>
 <wire x1="165.1" y1="2.54" x2="134.62" y2="2.54" width="0.1524" layer="91"/>
-<pinref part="J2" gate="G$1" pin="X34"/>
-<wire x1="165.1" y1="2.54" x2="187.96" y2="7.62" width="0.1524" layer="91"/>
-<junction x="165.1" y="2.54"/>
 <wire x1="134.62" y1="-22.86" x2="134.62" y2="2.54" width="0.1524" layer="91"/>
-<junction x="134.62" y="-22.86"/>
 </segment>
 <segment>
@@
 <wire x1="10.16" y1="71.12" x2="10.16" y2="66.04" width="0.1524" layer="91"/>
 </segment>
+<segment>
+<pinref part="SJ1" gate="1" pin="2"/>
+<pinref part="GND10" gate="1" pin="GND"/>
+<wire x1="157.48" y1="-33.02" x2="162.56" y2="-33.02" width="0.1524" layer="91"/>
+</segment>
+<segment>
+<pinref part="J2" gate="G$1" pin="X44"/>
+<wire x1="187.96" y1="-17.78" x2="182.88" y2="-17.78" width="0.1524" layer="91"/>
+<wire x1="182.88" y1="-17.78" x2="182.88" y2="-22.86" width="0.1524" layer="91"/>
+<wire x1="182.88" y1="-22.86" x2="187.96" y2="-22.86" width="0.1524" layer="91"/>
+<wire x1="187.96" y1="-22.86" x2="187.96" y2="-27.94" width="0.1524" layer="91"/>
+<pinref part="GND11" gate="1" pin="GND"/>
+<pinref part="SJ2" gate="1" pin="2"/>
+<wire x1="180.34" y1="-33.02" x2="187.96" y2="-33.02" width="0.1524" layer="91"/>
+<wire x1="187.96" y1="-33.02" x2="195.58" y2="-33.02" width="0.1524" layer="91"/>
+<wire x1="187.96" y1="-27.94" x2="187.96" y2="-33.02" width="0.1524" layer="91"/>
+<junction x="187.96" y="-33.02"/>
+</segment>
 </net>
 <net name="!RD" class="0">
@@
 </segment>
 </net>
+<net name="N$16" class="0">
+<segment>
+<pinref part="J1" gate="G$1" pin="X44"/>
+<pinref part="SJ1" gate="1" pin="1"/>
+<wire x1="165.1" y1="-22.86" x2="157.48" y2="-22.86" width="0.1524" layer="91"/>
+</segment>
+</net>
+<net name="N$17" class="0">
+<segment>
+<pinref part="J2" gate="G$1" pin="X34"/>
+<wire x1="187.96" y1="7.62" x2="180.34" y2="7.62" width="0.1524" layer="91"/>
+<wire x1="180.34" y1="7.62" x2="180.34" y2="5.08" width="0.1524" layer="91"/>
+<pinref part="SJ2" gate="1" pin="1"/>
+<wire x1="180.34" y1="5.08" x2="180.34" y2="-22.86" width="0.1524" layer="91"/>
+</segment>
+</net>

Commit message: Added Control Pad interface boards, updated board PDF, updated schematic PDF
Parts:
- added JP1, JP2: (no value), aquarius2:PINHD-1X10
- C9: value 10n -> 10nF
- Q1: value (none) -> 2N3904; device aq-transistor:-NPN-TO92L -> aq-transistor:2N3904
Connections:
- new net CPA-D00: JP1.5
- new net CPA-D01: JP1.4
- new net CPA-D02: JP1.2
- new net CPA-D03: JP1.1
- new net CPA-D04: JP1.6
- new net CPA-D05: JP1.8
- new net CPA-D06: JP1.10
- new net CPA-D07: JP1.9
- new net CPA-GND: JP1.3, JP1.7
- new net CPB-D00: JP2.5
- new net CPB-D01: JP2.4
- new net CPB-D02: JP2.2
- new net CPB-D03: JP2.1
- new net CPB-D04: JP2.6
- new net CPB-D05: JP2.8
- new net CPB-D06: JP2.10
- new net CPB-D07: JP2.9
- new net CPB-GND: JP2.3, JP2.7
Other:
- note added: "09 SEP 2020"
- note added: "Control Pad Interface Boards"
- note removed: "02 SEP 2020"
- moved on the sheet: R1, R2, R3
