File: eagle/mini_exp_v1-1-0c.brd (EAGLE design)
At the start: 208.6 x 112.5 mm, 34 parts, among them J1 CR22A-44D-2.54DS(70)STRAIGHT, J2 CR22A-44D-2.54DS(70)STRAIGHT, J3 DB9-MALE-RA, J4 DB9-MALE-RA, Q1 2N3904, U1 AY-3-8910, U2 74LS244N, U3 74LS244N, U4 74LS74N, U5 74LS30N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

Commit message: Added IO Header to Rev C
Parts:
- added JP3: (no value), aquarius2:2X10
- moved Q1 5.08 mm to (40.6, 18.8)
- moved R1 3.81 mm to (39.0, 25.0)
- moved R2 3.81 mm to (39.0, 28.9)
- moved R3 3.81 mm to (39.0, 32.8)
Connections:
- removed net N$100: J4.P$3, U1.7
- removed net N$101: J4.P$9, U1.10
- removed net N$102: J3.P$2, U1.14
- removed net N$103: J3.P$3, U1.15
- removed net N$104: J3.P$4, U1.16
- removed net N$105: J3.P$5, U1.17
- removed net N$106: J3.P$6, U1.21
- removed net N$107: J3.P$7, U1.20
- removed net N$108: J3.P$8, U1.19
- removed net N$109: J3.P$9, U1.18
- removed net N$18: J4.P$6, U1.13
- removed net N$94: J4.P$2, U1.6
- removed net N$95: J4.P$7, U1.12
- removed net N$96: J4.P$8, U1.11
- removed net N$98: J4.P$5, U1.9
- removed net N$99: J4.P$4, U1.8
- new net IOA0: J3.P$6, JP3.19, U1.21
- new net IOA1: J3.P$7, JP3.18, U1.20
- new net IOA2: J3.P$8, JP3.17, U1.19
- new net IOA3: J3.P$9, JP3.16, U1.18
- new net IOA4: J3.P$5, JP3.15, U1.17
- new net IOA5: J3.P$4, JP3.14, U1.16
- new net IOA6: J3.P$3, JP3.13, U1.15
- new net IOA7: J3.P$2, JP3.12, U1.14
- new net IOB0: J4.P$6, JP3.2, U1.13
- new net IOB1: J4.P$7, JP3.3, U1.12
- new net IOB2: J4.P$8, JP3.4, U1.11
- new net IOB3: J4.P$9, JP3.5, U1.10
- new net IOB4: J4.P$5, JP3.6, U1.9
- new net IOB5: J4.P$4, JP3.7, U1.8
- new net IOB6: J4.P$3, JP3.8, U1.7
- new net IOB7: J4.P$2, JP3.9, U1.6
- net GND: now also JP3.1, JP3.20
- net VCC: now also JP3.10, JP3.11
Routing:
- net GND: track 335.8 -> 434.3 mm, vias 16 -> 1
- net IOA2: track 0.00 -> 92.6 mm
- net IOB5: track 0.00 -> 91.6 mm
- net IOA0: track 0.00 -> 82.9 mm
- net IOB7: track 0.00 -> 75.7 mm
- net IOB0: track 0.00 -> 72.0 mm
- net IOB6: track 0.00 -> 68.2 mm
- net IOB1: track 0.00 -> 67.7 mm
- net N$106: track 65.0 -> 0.00 mm, vias 1 -> 0
- net IOB3: track 0.00 -> 63.7 mm
- net IOB2: track 0.00 -> 63.2 mm
- net IOB4: track 0.00 -> 59.8 mm
- net N$18: track 57.8 -> 0.00 mm, vias 1 -> 0
- net N$103: track 56.9 -> 0.00 mm, vias 1 -> 0
- net IOA1: track 0.00 -> 56.4 mm, vias 0 -> 1
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- added copper zone on layer 16, net N$18
- added copper zone on layer 16, net N$21
- added copper zone on layer 16, net N$22
- added copper zone on layer 16, net N$94
- added copper zone on layer 16, net N$95
- added copper zone on layer 16, net N$96
- added copper zone on layer 16, net N$98
- removed copper zone on layer 16, net N$209
- removed copper zone on layer 16, net N$225
- removed copper zone on layer 16, net N$228
- removed copper zone on layer 16, net N$231
- removed copper zone on layer 16, net N$237
- removed copper zone on layer 16, net N$240
- removed copper zone on layer 16, net N$243
- removed copper zone on layer 16, net N$247
- removed copper zone on layer 16, net N$255
- removed copper zone on layer 16, net N$257
- removed copper zone on layer 16, net N$260
- removed copper zone on layer 16, net N$282
- removed copper zone on layer 16, net N$288
- removed copper zone on layer 16, net N$300
- removed copper zone on layer 16, net N$302
- removed copper zone on layer 16, net N$311
- removed copper zone on layer 16, net N$321
- removed copper zone on layer 16, net N$332
- removed copper zone on layer 16, net N$338
- removed copper zone on layer 16, net N$352
Other:
- board text added: "AY-3-8910 I/O Header"
- board text added: "Expansion Bus Header"
- board text added: "IOA0"
- board text added: "IOA1"
- board text added: "IOA2"
- board text added: "IOA3"
- board text added: "IOA4"
- board text added: "IOA5"
- board text added: "IOA6"
- board text added: "IOA7"
- board text added: "IOB0"
- board text added: "IOB1"
- board text added: "IOB2"
- board text added: "IOB3"
- board text added: "IOB4"
- board text added: "IOB5"
- board text added: "IOB6"
- board text added: "IOB7"
