File: diy-control-pad/eagle/control_pad_v1-1-0x.brd (EAGLE design)
At the start: 68.6 x 138.4 mm, 64 parts, among them K1 TACT-SPST, K2 TACT-SPST, K3 TACT-SPST, K4 TACT-SPST, K5 TACT-SPST, K6 TACT-SPST, P1 TACT-SPST, P10 TACT-SPST, P11 TACT-SPST, P12 TACT-SPST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

Commit message: Post publishing clean up, Add Rev C
Connections:
- removed net N$4: P14.P$2, P14.P$4
- net GND: now also P14.P$2, P14.P$4
Routing:
- net N$4: track 7.55 -> 0.00 mm
- net GND: track 369.0 -> 376.4 mm
Other:
- board size 68.6 x 138.4 mm -> 68.6 x 137.8 mm
- board text added: "DIY Aquarius Control Pad by Sean P. Harrington, sph@1stage.com v1.1.0 Rev B - 19 OCT 2020"
- board text removed: "DIY Aquarius Control Pad by Sean P. Harrington, sph@1stage.com v1.1.0 Rev A - 11 OCT 2020"
Changed lines of the file:
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@@
 </layers>
 <board>
-<fusionsync huburn="a.cGVyc29uYWw6dWUyYWYyYWU4" projecturn="a.cGVyc29uYWw6dWUyYWYyYWU4IzIwMjAwODA5MzIyMjM1NDUx" f3durn="urn:adsk.wipprod:dm.lineage:Uy6oOUvdS5SKO7vhS9LsxA" pcbguid="5aefa80b-566f-4d0d-970b-879f518ca27a" lastpulledtime="" lastsyncedchangeguid="" latestrevisionid="c3bf1271-6840-4c2b-a01e-e2eef5b6c980" lastsyncedrevisionid="c3bf1271-6840-4c2b-a01e-e2eef5b6c980" lastboardhashguid="1537c16d-61dd-9f93-5075-3888f92f2155" lastpushedtime="2020-10-13T21:02:52Z" linktopcb3d="true"/>
+<fusionsync huburn="a.cGVyc29uYWw6dWUyYWYyYWU4" projecturn="a.cGVyc29uYWw6dWUyYWYyYWU4IzIwMjAwODA5MzIyMjM1NDUx" f3durn="urn:adsk.wipprod:dm.lineage:Uy6oOUvdS5SKO7vhS9LsxA" pcbguid="" lastpulledtime="" lastsyncedchangeguid="" latestrevisionid="c3bf1271-6840-4c2b-a01e-e2eef5b6c980" lastsyncedrevisionid="c3bf1271-6840-4c2b-a01e-e2eef5b6c980" lastboardhashguid="1537c16d-61dd-9f93-5075-3888f92f2155" lastpushedtime="2020-10-13T21:02:52Z" linktopcb3d="true"/>
 <plain>
 <wire x1="1.27" y1="0" x2="67.31" y2="0" width="0" layer="20"/>
@@
 <wire x1="20.32" y1="113.03" x2="24.13" y2="102.87" width="0.1524" layer="21"/>
 <wire x1="48.26" y1="113.03" x2="44.45" y2="102.87" width="0.1524" layer="21"/>
-<wire x1="26.67" y1="130.81" x2="41.91" y2="130.81" width="0" layer="20" curve="-180"/>
-<wire x1="30.48" y1="130.81" x2="38.1" y2="130.81" width="0" layer="20" curve="-180"/>
-<wire x1="38.1" y1="128.27" x2="30.48" y2="128.27" width="0" layer="20" curve="-180"/>
-<wire x1="30.48" y1="130.81" x2="30.48" y2="128.27" width="0" layer="20"/>
-<wire x1="38.1" y1="130.81" x2="38.1" y2="128.27" width="0" layer="20"/>
-<wire x1="41.91" y1="130.81" x2="67.31" y2="116.84" width="0" layer="20"/>
-<wire x1="26.67" y1="130.81" x2="1.27" y2="116.84" width="0" layer="20"/>
-<wire x1="43.18" y1="124.46" x2="43.18" y2="119.38" width="0" layer="20"/>
-<wire x1="25.4" y1="124.46" x2="25.4" y2="119.38" width="0" layer="20"/>
-<wire x1="29.21" y1="124.46" x2="29.21" y2="119.38" width="0" layer="20"/>
-<wire x1="39.37" y1="124.46" x2="39.37" y2="119.38" width="0" layer="20"/>
-<wire x1="25.4" y1="124.46" x2="29.21" y2="124.46" width="0" layer="20" curve="-180"/>
-<wire x1="39.37" y1="124.46" x2="43.18" y2="124.46" width="0" layer="20" curve="-180"/>
-<wire x1="43.18" y1="119.38" x2="39.37" y2="119.38" width="0" layer="20" curve="-180"/>
-<wire x1="29.21" y1="119.38" x2="25.4" y2="119.38" width="0" layer="20" curve="-180"/>
+<wire x1="38.1" y1="123.19" x2="30.48" y2="123.19" width="0" layer="20" curve="-180"/>
+<wire x1="30.48" y1="130.81" x2="30.48" y2="123.19" width="0" layer="20"/>
+<wire x1="38.1" y1="130.81" x2="38.1" y2="123.19" width="0" layer="20"/>
+<wire x1="41.91" y1="135.89" x2="67.31" y2="116.84" width="0" layer="20"/>
+<wire x1="26.67" y1="135.89" x2="1.27" y2="116.84" width="0" layer="20"/>
+<wire x1="44.45" y1="129.54" x2="44.45" y2="121.92" width="0" layer="20"/>
+<wire x1="24.13" y1="129.54" x2="24.13" y2="121.92" width="0" layer="20"/>
+<wire x1="27.94" y1="129.54" x2="27.94" y2="121.92" width="0" layer="20"/>
+<wire x1="40.64" y1="129.54" x2="40.64" y2="121.92" width="0" layer="20"/>
+<wire x1="24.13" y1="129.54" x2="27.94" y2="129.54" width="0" layer="20" curve="-180"/>
+<wire x1="40.64" y1="129.54" x2="44.45" y2="129.54" width="0" layer="20" curve="-180"/>
+<wire x1="44.45" y1="121.92" x2="40.64" y2="121.92" width="0" layer="20" curve="-180"/>
+<wire x1="27.94" y1="121.92" x2="24.13" y2="121.92" width="0" layer="20" curve="-180"/>
 <text x="34.29" y="115.824" size="1.27" layer="21" distance="40" align="center">Insert wires through upper holes corresponding
 with FEMALE plug position on your cable.</text>
@@
 <text x="63.5" y="88.9" size="1.27" layer="21" rot="R90" align="center">DIY Aquarius Control Pad
 by Sean P. Harrington, sph@1stage.com
-v1.1.0 Rev A - 11 OCT 2020</text>
+v1.1.0 Rev B - 19 OCT 2020</text>
 <text x="34.29" y="101.854" size="1.27" layer="21" distance="40" align="center">Solder wires to corresponding lower holes.</text>
+<wire x1="38.1" y1="135.89" x2="41.91" y2="135.89" width="0" layer="20" curve="-180"/>
+<wire x1="26.67" y1="135.89" x2="30.48" y2="135.89" width="0" layer="20" curve="-180"/>
+<wire x1="38.1" y1="135.89" x2="38.1" y2="130.81" width="0" layer="20"/>
+<wire x1="30.48" y1="135.89" x2="30.48" y2="130.81" width="0" layer="20"/>
 </plain>
 <attributes>
@@
 <wire x1="39.624" y1="14.859" x2="39.63845625" y2="14.944565625" width="0.508" layer="16"/>
 <wire x1="32.0294" y1="14.859" x2="31.877" y2="14.859" width="0.508" layer="16"/>
-<polygon width="0" layer="1" orphans="yes">
-<vertex x="0" y="116.84"/>
-<vertex x="26.67" y="130.81"/>
-<vertex x="26.67" y="137.16"/>
-<vertex x="34.29" y="139.7"/>
-<vertex x="41.91" y="137.16"/>
-<vertex x="41.91" y="130.81"/>
-<vertex x="68.58" y="116.84"/>
+<contactref element="P14" pad="P$2"/>
+<contactref element="P14" pad="P$4"/>
+<wire x1="44.097096875" y1="51.7886" x2="46.721540625" y2="54.41304375" width="0.508" layer="1"/>
+<wire x1="46.721540625" y1="54.41304375" x2="46.721540625" y2="58.124565625" width="0.508" layer="1"/>
+<polygon width="0.1524" layer="1" orphans="yes">
+<vertex x="0" y="115.57"/>
+<vertex x="30.48" y="138.43"/>
+<vertex x="38.1" y="138.43"/>
+<vertex x="68.58" y="115.57"/>
 <vertex x="68.58" y="0"/>
 <vertex x="0" y="0"/>
 </polygon>
-<polygon width="0" layer="16" orphans="yes">
-<vertex x="0" y="116.84"/>
-<vertex x="26.67" y="130.81"/>
-<vertex x="26.67" y="137.16"/>
-<vertex x="34.29" y="139.7"/>
-<vertex x="41.91" y="137.16"/>
-<vertex x="41.91" y="130.81"/>
-<vertex x="68.58" y="116.84"/>
+<polygon width="0.1524" layer="16" orphans="yes">
+<vertex x="0" y="115.57"/>
+<vertex x="30.48" y="138.43"/>
+<vertex x="38.1" y="138.43"/>
+<vertex x="68.58" y="115.57"/>
 <vertex x="68.58" y="0"/>
 <vertex x="0" y="0"/>
@@
 <wire x1="22.1234" y1="58.4454" x2="21.85845625" y2="58.124565625" width="0.508" layer="1"/>
 </signal>
-<signal name="N$4">
-<contactref element="P14" pad="P$4"/>
-<contactref element="P14" pad="P$2"/>
-<wire x1="44.2468" y1="55.8038" x2="44.2468" y2="51.8414" width="0.508" layer="1"/>
-<wire x1="46.5582" y1="58.1152" x2="44.2468" y2="55.8038" width="0.508" layer="1"/>
-<wire x1="44.2468" y1="51.8414" x2="44.097096875" y2="51.7886" width="0.508" layer="1"/>
-<wire x1="46.5582" y1="58.1152" x2="46.721540625" y2="58.124565625" width="0.508" layer="1"/>
-</signal>
 </signals>
