File: diy-control-pad/eagle/control_pad_v1-1-0x.sch (EAGLE design)
At the start: 64 parts, among them K1 TACT-SPST, K2 TACT-SPST, K3 TACT-SPST, K4 TACT-SPST, K5 TACT-SPST, K6 TACT-SPST, P1 TACT-SPST, P10 TACT-SPST, P11 TACT-SPST, P12 TACT-SPST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

Commit message: Post publishing clean up, Add Rev C
Connections:
- removed net N$4: P14.P$2
- net GND: now also P14.P$2
Changed lines of the file:
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@@
 <pinref part="P13" gate="G$1" pin="P$2"/>
+</segment>
+<segment>
+<pinref part="P14" gate="G$1" pin="P$2"/>
+<pinref part="GND3" gate="1" pin="GND"/>
+<wire x1="25.4" y1="58.42" x2="27.94" y2="58.42" width="0.1524" layer="91"/>
 </segment>
 </net>
@@
 </segment>
 </net>
-<net name="N$4" class="0">
-<segment>
-<wire x1="25.4" y1="58.42" x2="27.94" y2="58.42" width="0.1524" layer="91"/>
-<pinref part="GND3" gate="1" pin="GND"/>
-<pinref part="P14" gate="G$1" pin="P$2"/>
-</segment>
-</net>
